File: pcb/freaku4X/freaku4X.kicad_pcb (KiCad board)
At the start: 2 copper layers, 85 parts, among them SW1 RotaryEncoder_Switch, SW10 SW_SPST, SW11 SW_SPST, SW12 SW_SPST, SW13 SW_SPST, SW14 SW_SPST, SW15 SW_SPST, SW16 SW_SPST, SW17 SW_SPST, SW18 SW_SPST, SW19 SW_SPST, SW2 SW_SPST, SW20 SW_SPST, SW21 SW_SPST, SW22 SW_SPST, SW23 SW_SPST, SW24 SW_SPST, SW25 SW_SPST, SW26 SW_SPST, SW27 SW_SPST, SW28 SW_SPST, SW29 SW_SPST, SW3 SW_SPST, SW30 SW_SPST, SW31 SW_SPST, SW32 SW_SPST, SW33 SW_SPST, SW34 SW_SPST, SW35 SW_SPST, SW36 SW_SPST, SW37 SW_SPST, SW38 SW_SPST, SW39 SW_SPST, SW4 SW_SPST, SW40 SW_SPST, SW41 SW_SPST, SW42 SW_SPST, SW43 SW_SPST, SW5 SW_SPST, SW6 SW_SPST, SW7 SW_SPST, SW8 SW_SPST, SW9 SW_SPST, U1 ProMicro

Commit message: finish first iteration of PCB
Parts:
- added H1: MountingHole, MountingHole:MountingHole_2.2mm_M2, F.Cu at (188.9, 65.9)
- added H2: MountingHole, MountingHole:MountingHole_2.2mm_M2, F.Cu at (169.9, 50.0)
- added H2: MountingHole, MountingHole:MountingHole_2.2mm_M2, F.Cu at (131.8, 50.0)
- added H2: MountingHole, MountingHole:MountingHole_2.2mm_M2, F.Cu at (112.7, 65.9)
- added H3: MountingHole, MountingHole:MountingHole_2.2mm_M2, F.Cu at (74.6, 85.7)
- added H4: MountingHole, MountingHole:MountingHole_2.2mm_M2, F.Cu at (227.0, 85.7)
- added H5: MountingHole, MountingHole:MountingHole_2.2mm_M2, F.Cu at (131.8, 104.8)
- added H6: MountingHole, MountingHole:MountingHole_2.2mm_M2, F.Cu at (169.9, 104.8)
- added H7: MountingHole, MountingHole:MountingHole_2.2mm_M2, F.Cu at (74.6, 123.8)
- added H8: MountingHole, MountingHole:MountingHole_2.2mm_M2, F.Cu at (227.0, 123.8)
- added REF**: Stabilizer_MX_2u, keyswitches:Stabilizer_MX_2u, F.Cu at (150.8, 133.3)
- added SW44: SW_SPST, keyswitches:SW_MX, F.Cu at (150.8, 133.3)
- D1, D10, D11, D12, D13, D14, D15, D16, D17, D18, D19, D2, D20, D21, D22, D23, D24, D25, D26, D27, D28, D29, D3, D30, D31, D32, D33, D34, D35, D36, D37, D38, D39, D4, D40, D5, D6, D7, D8, D9: footprint kbd:D3_TH_SMD_v2 -> Keebio-Parts:Diode-dual; moved to B.Cu
- SW42: moved to B.Cu
- moved D31 269.0 mm to (65.1, 141.3), turned to 180 degrees
- moved D37 262.0 mm to (122.2, 141.3), turned to 180 degrees
- moved D35 253.5 mm to (217.5, 141.3), turned to 180 degrees
- moved D34 243.0 mm to (179.4, 141.3), turned to 180 degrees
- moved D24 227.2 mm to (179.4, 123.0), turned to 180 degrees
- moved D25 215.1 mm to (217.5, 123.0), turned to 180 degrees
- moved D40 213.9 mm to (236.5, 141.3), turned to 180 degrees
- moved D7 212.9 mm to (122.2, 86.5), turned to 180 degrees
- moved D5 200.4 mm to (218.1, 84.9), turned to 180 degrees
- moved D20 200.0 mm to (236.5, 105.6), turned to 180 degrees
- moved D9 191.6 mm to (198.4, 86.5), turned to 180 degrees
- moved D32 189.8 mm to (103.2, 141.3), turned to 180 degrees
- moved D29 189.3 mm to (198.4, 124.6), turned to 180 degrees
- moved D15 188.5 mm to (217.5, 104.0), turned to 180 degrees
- moved D10 187.9 mm to (236.5, 86.5), turned to 180 degrees
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Connections:
- U1 pad 13: col1 -> col5
- U1 pad 14: col2 -> col4
- U1 pad 16: col4 -> col2
- U1 pad 17: col5 -> col1
Routing:
- net col5: track 0.00 -> 339.5 mm, vias 0 -> 6
- net col4: track 0.00 -> 305.8 mm, vias 0 -> 6
- net col3: track 0.00 -> 288.2 mm, vias 0 -> 6
- net row8: track 0.00 -> 282.8 mm, vias 0 -> 2
- net row7: track 0.00 -> 262.9 mm, vias 0 -> 2
- net row6: track 0.00 -> 250.2 mm, vias 0 -> 5
- net col2: track 0.00 -> 239.2 mm, vias 0 -> 7
- net row5: track 0.00 -> 235.0 mm, vias 0 -> 1
- net row4: track 0.00 -> 221.6 mm, vias 0 -> 1
- net col1: track 0.00 -> 217.9 mm, vias 0 -> 5
- net row3: track 0.00 -> 215.2 mm, vias 0 -> 5
- net gnd: track 0.00 -> 201.7 mm, vias 0 -> 4
- net row2: track 0.00 -> 200.2 mm, vias 0 -> 2
- net row1: track 0.00 -> 194.0 mm, vias 0 -> 1
- net padA: track 0.00 -> 178.5 mm, vias 0 -> 2
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Other:
- board outline added: 190.5 x 95.2 mm
- board text added: "44 6F 20 79 6F 75 20 74 68 69 6E 6B 20 47 6F 64 20 73 74 61 79 73 20 69 6E 20 68 65 61 76 65 6E 20 62 65 63 61 75 73 65 20 68 65 20 74 6F 6F 20 6C 69 76 65 73 20 69 6E 20 66 65 61 72 20 6F 66 20 77 68 61 74 20 68 65 27 73 20 63 72 65 61 74 65 64 3F"
- board text added: "PCBPCBPCB"
- board text added: "by sporewoh"
- board text added: "freak out!"
- board text added: "freaku4X v0.1"
- board text added: "place pro-micro here"
- board text added: "{dblquote}You cheated not only the game, but yourself. You didn't grow. You didn't improve. You took a shortcut and gained nothing. You experienced a hollow victory. Nothing was risked and nothing was gained. It's sad you don't know the difference.{dblquote} - Sun Tzu"
