File: pcb/freaku4X/freaku4X.kicad_sch (KiCad schematic)
At the start: 85 parts, among them SW10 SW_SPST, SW11 SW_SPST, SW12 SW_SPST, SW13 SW_SPST, SW14 SW_SPST, SW15 SW_SPST, SW16 SW_SPST, SW17 SW_SPST, SW18 SW_SPST, SW19 SW_SPST, SW20 SW_SPST, SW21 SW_SPST, SW22 SW_SPST, SW23 SW_SPST, SW24 SW_SPST, SW25 SW_SPST, SW26 SW_SPST, SW27 SW_SPST, SW28 SW_SPST, SW29 SW_SPST, SW3 SW_SPST, SW30 SW_SPST, SW31 SW_SPST, SW32 SW_SPST, SW33 SW_SPST, SW34 SW_SPST, SW35 SW_SPST, SW36 SW_SPST, SW37 SW_SPST, SW38 SW_SPST, SW39 SW_SPST, SW4 SW_SPST, SW40 SW_SPST, SW41 SW_SPST, SW5 SW_SPST, SW6 SW_SPST, SW7 SW_SPST, SW8 SW_SPST, SW9 SW_SPST

Commit message: finish first iteration of PCB
Parts:
- added H1, H2, H3, H4, H5, H6, H7, H8: MountingHole, MountingHole:MountingHole_2.2mm_M2, symbol Mechanical:MountingHole
- added SW44: SW_SPST, keyswitches:SW_MX, symbol Switch:SW_SPST
- D1: value (none) -> 1N4148
- OL1: value (none) -> OLED; footprint (none) -> kbd:OLED_v2
- SW1: value (none) -> RotaryEncoder_Switch; footprint (none) -> Rotary_Encoder:RotaryEncoder_Alps_EC11E-Switch_Vertical_H20mm
- SW10, SW11, SW12, SW13, SW14, SW15, SW16, SW17, SW18, SW19, SW20, SW21, SW22, SW23, SW24, SW25, SW26, SW27, SW28, SW29, SW3, SW30, SW31, SW32, SW33, SW34, SW35, SW36, SW37, SW38, SW39, SW4, SW40, SW41, SW5, SW6, SW7, SW8, SW9: footprint (none) -> keyswitches:Kailh_socket_MX_optional
- SW2: value (none) -> SW_SPST; footprint (none) -> keyswitches:Kailh_socket_MX_optional
- SW42: value (none) -> SW_SPST; footprint (none) -> kbd:ResetSW_4
- SW43: value (none) -> SW_SPST; footprint (none) -> kbd:ResetSW
- U1: value (none) -> ProMicro; footprint (none) -> kbd:ProMicro_v3
Connections:
- net col1: now also U1.17 (A0/PF7); no longer U1.13 (10/PB6)
- net col2: now also U1.16 (15/PB1); no longer U1.14 (16/PB2)
- net col3: now also SW44.2 (B)
- net col4: now also U1.14 (16/PB2); no longer U1.16 (15/PB1)
- net col5: now also U1.13 (10/PB6); no longer U1.17 (A0/PF7)
- net at D33.2 (A), SW36.1 (A): now also SW44.1 (A)
